File: relay_interlock.sch (KiCad schematic (older format))
At the start: 6 parts

Commit message: Rough Draft of Relay Circuit
Parts:
- removed D? (x2): LED, symbol Device:LED
- removed SW?: SW_Push, symbol Switch:SW_Push
- removed U?: 74AUC2G08, symbol 74xGxx:74AUC2G08
- removed U?: 74AHC1G08, symbol 74xGxx:74AHC1G08
- added D? (x2): LTST-C150KRKT, digikey-footprints:1206, symbol dk_LED-Indication-Discrete:LTST-C150KRKT
- added D?: LTST-C150KGKT, digikey-footprints:1206, symbol dk_LED-Indication-Discrete:LTST-C150KGKT
- added Q? (x2): BSS138W, SOT323-R, symbol BSS138W:BSS138W
- added R?: 100k, symbol Device:R
- added R? (x3): 500, symbol Device:R
- added U?: SN74LVC1G08DCKR, digikey-footprints:SC-70-5, symbol dk_Logic-Gates-and-Inverters:SN74LVC1G08DCKR
- added U?: SN74LVC1G14DCKR, DCK5, symbol 2020-06-28_23-59-59:SN74LVC1G14DCKR
- added U?: SR4D4005, RELAY10-5MM-6.5MM, symbol 2020-06-26_17-54-09:SR4D4005
Connections:
- net labels added: +5VOut1, Enable_Conn_1, Enable_Conn_2, ErrSig1, GND
- wire segments 0 -> 49
- no-connect marks 0 -> 3
Other:
- moved on the sheet: SW?

Commit message: Made 5V local label to each sheet
Connections:
- net +5VOut1 renamed +5Vin
Changed lines of the file:
@@
 $Descr A4 11693 8268
 encoding utf-8
-Sheet 2 3
+Sheet 2 2
 Title ""
 Date ""
@@
 	0    1    1    0
 $EndComp
-Text GLabel 3750 3350 0    50   Input ~ 0
-+5VOut1
 Wire Wire Line
 	6100 2650 5800 2650
 $Comp
-L power:GND #PWR?
+L power:GND #PWR0107
 U 1 1 5EFC1523
 P 6700 2650
-F 0 "#PWR?" H 6700 2400 50  0001 C CNN
+F 0 "#PWR0107" H 6700 2400 50  0001 C CNN
 F 1 "GND" H 6705 2477 50  0000 C CNN
 F 2 "" H 6700 2650 50  0001 C CNN
@@
 Wire Wire Line
 	3700 2650 4000 2650
-Text GLabel 2800 2650 0    50   Input ~ 0
-+5VOut1
-Wire Wire Line
-	2800 2650 3000 2650
 Wire Wire Line
 	3700 3200 3700 2650
@@
 	3400 2650 3700 2650
 Connection ~ 3700 2650
-Text GLabel 3300 2850 0    50   Input ~ 0
-+5VOut1
-Wire Wire Line
-	3300 2850 4000 2850
 $Comp
 L dk_LED-Indication-Discrete:LTST-C150KRKT D?
@@
 	1800 3000 2100 3000
 $Comp
-L power:GND #PWR?
+L power:GND #PWR0108
 U 1 1 5EFD6108
 P 1800 3550
-F 0 "#PWR?" H 1800 3300 50  0001 C CNN
+F 0 "#PWR0108" H 1800 3300 50  0001 C CNN
 F 1 "GND" H 1805 3377 50  0000 C CNN
 F 2 "" H 1800 3550 50  0001 C CNN
@@
 $EndComp
 Wire Wire Line
-	3750 3350 4000 3350
-Wire Wire Line
 	3700 3200 3300 3200
 Wire Wire Line
@@
 	2500 3450 2500 3700
 $Comp
-L power:GND #PWR?
+L power:GND #PWR0109
 U 1 1 5EFDD582
 P 2500 4200
-F 0 "#PWR?" H 2500 3950 50  0001 C CNN
+F 0 "#PWR0109" H 2500 3950 50  0001 C CNN
 F 1 "GND" H 2505 4027 50  0000 C CNN
 F 2 "" H 2500 4200 50  0001 C CNN
@@
 	3050 3450 2800 3450
 $Comp
-L power:GND #PWR?
+L power:GND #PWR0110
 U 1 1 5EFA4E4F
 P 3050 4300
-F 0 "#PWR?" H 3050 4050 50  0001 C CNN
+F 0 "#PWR0110" H 3050 4050 50  0001 C CNN
 F 1 "GND" H 3055 4127 50  0000 C CNN
 F 2 "" H 3050 4300 50  0001 C CNN
@@
 Wire Wire Line
 	3050 4300 3050 4050
-Text GLabel 5500 4050 1    50   Input ~ 0
-+5VOut1
-Wire Wire Line
-	5500 4050 5500 4200
-$Comp
-L power:GND #PWR?
+$Comp
+L power:GND #PWR0111
 U 1 1 5EFA6D3C
 P 5500 5000
-F 0 "#PWR?" H 5500 4750 50  0001 C CNN
+F 0 "#PWR0111" H 5500 4750 50  0001 C CNN
 F 1 "GND" H 5505 4827 50  0000 C CNN
 F 2 "" H 5500 5000 50  0001 C CNN
@@
 	1    0    0    -1
 $EndComp
-Text GLabel 5700 5700 2    50   Input ~ 0
-+5VOut1
-Wire Wire Line
-	5700 5700 5400 5700
-$Comp
-L power:GND #PWR?
+$Comp
+L power:GND #PWR0112
 U 1 1 5EFB4DC8
 P 5700 5900
-F 0 "#PWR?" H 5700 5650 50  0001 C CNN
+F 0 "#PWR0112" H 5700 5650 50  0001 C CNN
 F 1 "GND" H 5705 5727 50  0000 C CNN
 F 2 "" H 5700 5900 50  0001 C CNN
@@
 $EndComp
 $Comp
-L power:GND #PWR?
+L power:GND #PWR0113
 U 1 1 5EFBA4E9
 P 7350 4750
-F 0 "#PWR?" H 7350 4500 50  0001 C CNN
+F 0 "#PWR0113" H 7350 4500 50  0001 C CNN
 F 1 "GND" H 7355 4577 50  0000 C CNN
 F 2 "" H 7350 4750 50  0001 C CNN
@@
 	1    0    0    -1
 $EndComp
-Text GLabel 7350 2850 1    50   Input ~ 0
-+5VOut1
-Wire Wire Line
-	7350 2850 7350 3200
 Wire Wire Line
 	7350 4000 7350 4150
 Wire Wire Line
 	7350 3500 7350 3700
+Text HLabel 7350 2600 1    50   Input ~ 0
++5Vin
+Wire Wire Line
+	7350 2600 7350 3200
+Text HLabel 2650 2650 0    50   Input ~ 0
++5Vin
+Wire Wire Line
+	2650 2650 3000 2650
+Text HLabel 3100 2850 0    50   Input ~ 0
++5Vin
+Wire Wire Line
+	3100 2850 4000 2850
+Text HLabel 3600 3350 0    50   Input ~ 0
++5Vin
+Wire Wire Line
+	3600 3350 4000 3350
+Text HLabel 5500 3900 1    50   Input ~ 0
++5Vin
+Wire Wire Line
+	5500 3900 5500 4200
+Text HLabel 6000 5700 2    50   Input ~ 0
++5Vin
+Wire Wire Line
+	5400 5700 6000 5700
 $EndSCHEMATC

Commit message: Annotations
Parts:
- gave numbers to parts that had none: 13
Changed lines of the file:
@@
 $Descr A4 11693 8268
 encoding utf-8
-Sheet 2 2
+Sheet 2 3
 Title ""
 Date ""
@@
 $EndDescr
 $Comp
-L Switch:SW_Push SW?
+L Switch:SW_Push SW301
 U 1 1 5EF5F5C0
 P 3200 2650
-F 0 "SW?" H 3200 2935 50  0000 C CNN
+AR Path="/5EF588A2/5EF5F5C0" Ref="SW301"  Part="1"
+AR Path="/5EFCF919/5EF5F5C0" Ref="SW201"  Part="1"
+F 0 "SW201" H 3200 2935 50  0000 C CNN
 F 1 "SW_Push" H 3200 2844 50  0000 C CNN
 F 2 "" H 3200 2850 50  0001 C CNN
@@
 $EndComp
 $Comp
-L BSS138W:BSS138W Q?
+L BSS138W:BSS138W Q301
 U 1 1 5EFBAF07
 P 6300 2650
-F 0 "Q?" V 6443 2650 50  0000 C CNN
+AR Path="/5EF588A2/5EFBAF07" Ref="Q301"  Part="1"
+AR Path="/5EFCF919/5EFBAF07" Ref="Q201"  Part="1"
+F 0 "Q201" V 6443 2650 50  0000 C CNN
 F 1 "BSS138W" V 6534 2650 50  0000 C CNN
 F 2 "SOT323-R" H 6300 2650 50  0001 L BNN
@@
 U 1 1 5EFC1523
 P 6700 2650
-F 0 "#PWR0107" H 6700 2400 50  0001 C CNN
+AR Path="/5EF588A2/5EFC1523" Ref="#PWR0107"  Part="1"
+AR Path="/5EFCF919/5EFC1523" Ref="#PWR0115"  Part="1"
+F 0 "#PWR0115" H 6700 2400 50  0001 C CNN
 F 1 "GND" H 6705 2477 50  0000 C CNN
 F 2 "" H 6700 2650 50  0001 C CNN
@@
 AR Path="/5EFBABE7" Ref="U?"  Part="1"
 AR Path="/5EF82676/5EFBABE7" Ref="U?"  Part="1"
-AR Path="/5EF588A2/5EFBABE7" Ref="U?"  Part="1"
-F 0 "U?" H 4900 3138 60  0000 C CNN
+AR Path="/5EF588A2/5EFBABE7" Ref="U302"  Part="1"
+AR Path="/5EFCF919/5EFBABE7" Ref="U202"  Part="1"
+F 0 "U202" H 4900 3138 60  0000 C CNN
 F 1 "SR4D4005" H 4900 3032 60  0000 C CNN
 F 2 "RELAY10-5MM-6.5MM" H 4900 2990 60  0001 C CNN
@@
 Connection ~ 3700 2650
 $Comp
-L dk_LED-Indication-Discrete:LTST-C150KRKT D?
+L dk_LED-Indication-Discrete:LTST-C150KRKT D301
 U 1 1 5EFD24D7
 P 2200 3000
-F 0 "D?" H 2150 2753 60  0000 C CNN
+AR Path="/5EF588A2/5EFD24D7" Ref="D301"  Part="1"
+AR Path="/5EFCF919/5EFD24D7" Ref="D201"  Part="1"
+F 0 "D201" H 2150 2753 60  0000 C CNN
 F 1 "LTST-C150KRKT" H 2150 2859 60  0000 C CNN
 F 2 "digikey-footprints:1206" H 2400 3200 60  0001 L CNN
@@
 	2400 3000 4000 3000
 $Comp
-L Device:R R?
+L Device:R R301
 U 1 1 5EFD53B2
 P 1800 3150
-F 0 "R?" H 1870 3196 50  0000 L CNN
+AR Path="/5EF588A2/5EFD53B2" Ref="R301"  Part="1"
+AR Path="/5EFCF919/5EFD53B2" Ref="R201"  Part="1"
+F 0 "R201" H 1870 3196 50  0000 L CNN
 F 1 "500" H 1870 3105 50  0000 L CNN
 F 2 "" V 1730 3150 50  0001 C CNN
@@
 U 1 1 5EFD6108
 P 1800 3550
-F 0 "#PWR0108" H 1800 3300 50  0001 C CNN
+AR Path="/5EF588A2/5EFD6108" Ref="#PWR0108"  Part="1"
+AR Path="/5EFCF919/5EFD6108" Ref="#PWR0116"  Part="1"
+F 0 "#PWR0116" H 1800 3300 50  0001 C CNN
 F 1 "GND" H 1805 3377 50  0000 C CNN
 F 2 "" H 1800 3550 50  0001 C CNN
@@
 	1800 3550 1800 3300
 $Comp
-L dk_LED-Indication-Discrete:LTST-C150KGKT D?
+L dk_LED-Indication-Discrete:LTST-C150KGKT D302
 U 1 1 5EFD7D41
 P 2600 3450
-F 0 "D?" H 2550 3203 60  0000 C CNN
+AR Path="/5EF588A2/5EFD7D41" Ref="D302"  Part="1"
+AR Path="/5EFCF919/5EFD7D41" Ref="D202"  Part="1"
+F 0 "D202" H 2550 3203 60  0000 C CNN
 F 1 "LTST-C150KGKT" H 2550 3309 60  0000 C CNN
 F 2 "digikey-footprints:1206" H 2800 3650 60  0001 L CNN
@@
 Connection ~ 3700 3200
 $Comp
-L Device:R R?
+L Device:R R302
 U 1 1 5EFDCB0F
 P 2500 3850
-F 0 "R?" H 2570 3896 50  0000 L CNN
+AR Path="/5EF588A2/5EFDCB0F" Ref="R302"  Part="1"
+AR Path="/5EFCF919/5EFDCB0F" Ref="R202"  Part="1"
+F 0 "R202" H 2570 3896 50  0000 L CNN
 F 1 "500" H 2570 3805 50  0000 L CNN
 F 2 "" V 2430 3850 50  0001 C CNN
@@
 U 1 1 5EFDD582
 P 2500 4200
-F 0 "#PWR0109" H 2500 3950 50  0001 C CNN
+AR Path="/5EF588A2/5EFDD582" Ref="#PWR0109"  Part="1"
+AR Path="/5EFCF919/5EFDD582" Ref="#PWR0117"  Part="1"
+F 0 "#PWR0117" H 2500 3950 50  0001 C CNN
 F 1 "GND" H 2505 4027 50  0000 C CNN
 F 2 "" H 2500 4200 50  0001 C CNN
@@
 	2500 4200 2500 4000
 $Comp
-L dk_Logic-Gates-and-Inverters:SN74LVC1G08DCKR U?
+L dk_Logic-Gates-and-Inverters:SN74LVC1G08DCKR U303
 U 1 1 5EF92FF9
 P 5500 4500
-F 0 "U?" H 5844 4553 60  0000 L CNN
+AR Path="/5EF588A2/5EF92FF9" Ref="U303"  Part="1"
+AR Path="/5EFCF919/5EF92FF9" Ref="U203"  Part="1"
+F 0 "U203" H 5844 4553 60  0000 L CNN
 F 1 "SN74LVC1G08DCKR" H 5844 4447 60  0000 L CNN
 F 2 "digikey-footprints:SC-70-5" H 5700 4700 60  0001 L CNN
@@
 	3300 3200 3150 3200
 $Comp
-L Device:R R?
+L Device:R R303
 U 1 1 5EFA444C
 P 3050 3900
-F 0 "R?" H 3120 3946 50  0000 L CNN
+AR Path="/5EF588A2/5EFA444C" Ref="R303"  Part="1"
+AR Path="/5EFCF919/5EFA444C" Ref="R203"  Part="1"
+F 0 "R203" H 3120 3946 50  0000 L CNN
 F 1 "100k" H 3120 3855 50  0000 L CNN
 F 2 "" V 2980 3900 50  0001 C CNN
@@
 U 1 1 5EFA4E4F
 P 3050 4300
-F 0 "#PWR0110" H 3050 4050 50  0001 C CNN
+AR Path="/5EF588A2/5EFA4E4F" Ref="#PWR0110"  Part="1"
+AR Path="/5EFCF919/5EFA4E4F" Ref="#PWR0118"  Part="1"
+F 0 "#PWR0118" H 3050 4050 50  0001 C CNN
 F 1 "GND" H 3055 4127 50  0000 C CNN
 F 2 "" H 3050 4300 50  0001 C CNN
@@
 U 1 1 5EFA6D3C
 P 5500 5000
-F 0 "#PWR0111" H 5500 4750 50  0001 C CNN
+AR Path="/5EF588A2/5EFA6D3C" Ref="#PWR0111"  Part="1"
+AR Path="/5EFCF919/5EFA6D3C" Ref="#PWR0119"  Part="1"
+F 0 "#PWR0119" H 5500 4750 50  0001 C CNN
 F 1 "GND" H 5505 4827 50  0000 C CNN
 F 2 "" H 5500 5000 50  0001 C CNN
@@
 	5850 4500 5800 4500
 $Comp
-L 2020-06-28_23-59-59:SN74LVC1G14DCKR U?
+L 2020-06-28_23-59-59:SN74LVC1G14DCKR U301
 U 1 1 5EFB2E9F
 P 3200 5700
-F 0 "U?" H 4300 6087 60  0000 C CNN
+AR Path="/5EF588A2/5EFB2E9F" Ref="U301"  Part="1"
+AR Path="/5EFCF919/5EFB2E9F" Ref="U201"  Part="1"
+F 0 "U201" H 4300 6087 60  0000 C CNN
 F 1 "SN74LVC1G14DCKR" H 4300 5981 60  0000 C CNN
 F 2 "DCK5" H 4300 5940 60  0001 C CNN
@@
 U 1 1 5EFB4DC8
 P 5700 5900
-F 0 "#PWR0112" H 5700 5650 50  0001 C CNN
+AR Path="/5EF588A2/5EFB4DC8" Ref="#PWR0112"  Part="1"
+AR Path="/5EFCF919/5EFB4DC8" Ref="#PWR0120"  Part="1"
+F 0 "#PWR0120" H 5700 5650 50  0001 C CNN
 F 1 "GND" H 5705 5727 50  0000 C CNN
 F 2 "" H 5700 5900 50  0001 C CNN
@@
 	4700 5300 5500 5300
 $Comp
-L BSS138W:BSS138W Q?
+L BSS138W:BSS138W Q302
 U 1 1 5EFB94AA
 P 7350 4350
-F 0 "Q?" V 7493 4350 50  0000 C CNN
+AR Path="/5EF588A2/5EFB94AA" Ref="Q302"  Part="1"
+AR Path="/5EFCF919/5EFB94AA" Ref="Q202"  Part="1"
+F 0 "Q202" V 7493 4350 50  0000 C CNN
 F 1 "BSS138W" V 7584 4350 50  0000 C CNN
 F 2 "SOT323-R" H 7350 4350 50  0001 L BNN
@@
 U 1 1 5EFBA4E9
 P 7350 4750
-F 0 "#PWR0113" H 7350 4500 50  0001 C CNN
+AR Path="/5EF588A2/5EFBA4E9" Ref="#PWR0113"  Part="1"
+AR Path="/5EFCF919/5EFBA4E9" Ref="#PWR0121"  Part="1"
+F 0 "#PWR0121" H 7350 4500 50  0001 C CNN
 F 1 "GND" H 7355 4577 50  0000 C CNN
 F 2 "" H 7350 4750 50  0001 C CNN
@@
 	7350 4750 7350 4550
 $Comp
-L dk_LED-Indication-Discrete:LTST-C150KRKT D?
+L dk_LED-Indication-Discrete:LTST-C150KRKT D303
 U 1 1 5EFBB268
 P 7350 3900
-F 0 "D?" H 7300 3653 60  0000 C CNN
+AR Path="/5EF588A2/5EFBB268" Ref="D303"  Part="1"
+AR Path="/5EFCF919/5EFBB268" Ref="D203"  Part="1"
+F 0 "D203" H 7300 3653 60  0000 C CNN
 F 1 "LTST-C150KRKT" H 7300 3759 60  0000 C CNN
 F 2 "digikey-footprints:1206" H 7550 4100 60  0001 L CNN
@@
 $EndComp
 $Comp
-L Device:R R?
+L Device:R R304
 U 1 1 5EFBC18E
 P 7350 3350
-F 0 "R?" H 7420 3396 50  0000 L CNN
+AR Path="/5EF588A2/5EFBC18E" Ref="R304"  Part="1"
+AR Path="/5EFCF919/5EFBC18E" Ref="R204"  Part="1"
+F 0 "R204" H 7420 3396 50  0000 L CNN
 F 1 "500" H 7420 3305 50  0000 L CNN
 F 2 "" V 7280 3350 50  0001 C CNN

Commit message: Bypass everything and run Error Check
Parts:
- added C301: 0.1u, symbol Device:C
- R301, R302, R304: value 500 -> 1k
Connections:
- net +5Vin: now also C301.2
- net GND: now also C301.1
Other:
- moved on the sheet: U301
Changed lines of the file:
@@
 $Descr A4 11693 8268
 encoding utf-8
-Sheet 2 3
+Sheet 3 3
 Title ""
 Date ""
@@
 AR Path="/5EF588A2/5EF5F5C0" Ref="SW301"  Part="1"
 AR Path="/5EFCF919/5EF5F5C0" Ref="SW201"  Part="1"
-F 0 "SW201" H 3200 2935 50  0000 C CNN
+F 0 "SW301" H 3200 2935 50  0000 C CNN
 F 1 "SW_Push" H 3200 2844 50  0000 C CNN
 F 2 "" H 3200 2850 50  0001 C CNN
@@
 AR Path="/5EF588A2/5EFBAF07" Ref="Q301"  Part="1"
 AR Path="/5EFCF919/5EFBAF07" Ref="Q201"  Part="1"
-F 0 "Q201" V 6443 2650 50  0000 C CNN
+F 0 "Q301" V 6443 2650 50  0000 C CNN
 F 1 "BSS138W" V 6534 2650 50  0000 C CNN
 F 2 "SOT323-R" H 6300 2650 50  0001 L BNN
@@
 AR Path="/5EF588A2/5EFC1523" Ref="#PWR0107"  Part="1"
 AR Path="/5EFCF919/5EFC1523" Ref="#PWR0115"  Part="1"
-F 0 "#PWR0115" H 6700 2400 50  0001 C CNN
+F 0 "#PWR0107" H 6700 2400 50  0001 C CNN
 F 1 "GND" H 6705 2477 50  0000 C CNN
 F 2 "" H 6700 2650 50  0001 C CNN
@@
 AR Path="/5EF588A2/5EFBABE7" Ref="U302"  Part="1"
 AR Path="/5EFCF919/5EFBABE7" Ref="U202"  Part="1"
-F 0 "U202" H 4900 3138 60  0000 C CNN
+F 0 "U302" H 4900 3138 60  0000 C CNN
 F 1 "SR4D4005" H 4900 3032 60  0000 C CNN
 F 2 "RELAY10-5MM-6.5MM" H 4900 2990 60  0001 C CNN
@@
 AR Path="/5EF588A2/5EFD24D7" Ref="D301"  Part="1"
 AR Path="/5EFCF919/5EFD24D7" Ref="D201"  Part="1"
-F 0 "D201" H 2150 2753 60  0000 C CNN
+F 0 "D301" H 2150 2753 60  0000 C CNN
 F 1 "LTST-C150KRKT" H 2150 2859 60  0000 C CNN
 F 2 "digikey-footprints:1206" H 2400 3200 60  0001 L CNN
@@
 AR Path="/5EF588A2/5EFD53B2" Ref="R301"  Part="1"
 AR Path="/5EFCF919/5EFD53B2" Ref="R201"  Part="1"
-F 0 "R201" H 1870 3196 50  0000 L CNN
-F 1 "500" H 1870 3105 50  0000 L CNN
+F 0 "R301" H 1870 3196 50  0000 L CNN
+F 1 "1k" H 1870 3105 50  0000 L CNN
 F 2 "" V 1730 3150 50  0001 C CNN
 F 3 "~" H 1800 3150 50  0001 C CNN
@@
 AR Path="/5EF588A2/5EFD6108" Ref="#PWR0108"  Part="1"
 AR Path="/5EFCF919/5EFD6108" Ref="#PWR0116"  Part="1"
-F 0 "#PWR0116" H 1800 3300 50  0001 C CNN
+F 0 "#PWR0108" H 1800 3300 50  0001 C CNN
 F 1 "GND" H 1805 3377 50  0000 C CNN
 F 2 "" H 1800 3550 50  0001 C CNN
@@
 AR Path="/5EF588A2/5EFD7D41" Ref="D302"  Part="1"
 AR Path="/5EFCF919/5EFD7D41" Ref="D202"  Part="1"
-F 0 "D202" H 2550 3203 60  0000 C CNN
+F 0 "D302" H 2550 3203 60  0000 C CNN
 F 1 "LTST-C150KGKT" H 2550 3309 60  0000 C CNN
 F 2 "digikey-footprints:1206" H 2800 3650 60  0001 L CNN
@@
 AR Path="/5EF588A2/5EFDCB0F" Ref="R302"  Part="1"
 AR Path="/5EFCF919/5EFDCB0F" Ref="R202"  Part="1"
-F 0 "R202" H 2570 3896 50  0000 L CNN
-F 1 "500" H 2570 3805 50  0000 L CNN
+F 0 "R302" H 2570 3896 50  0000 L CNN
+F 1 "1k" H 2570 3805 50  0000 L CNN
 F 2 "" V 2430 3850 50  0001 C CNN
 F 3 "~" H 2500 3850 50  0001 C CNN
@@
 AR Path="/5EF588A2/5EFDD582" Ref="#PWR0109"  Part="1"
 AR Path="/5EFCF919/5EFDD582" Ref="#PWR0117"  Part="1"
-F 0 "#PWR0117" H 2500 3950 50  0001 C CNN
+F 0 "#PWR0109" H 2500 3950 50  0001 C CNN
 F 1 "GND" H 2505 4027 50  0000 C CNN
 F 2 "" H 2500 4200 50  0001 C CNN
@@
 AR Path="/5EF588A2/5EF92FF9" Ref="U303"  Part="1"
 AR Path="/5EFCF919/5EF92FF9" Ref="U203"  Part="1"
-F 0 "U203" H 5844 4553 60  0000 L CNN
+F 0 "U303" H 5844 4553 60  0000 L CNN
 F 1 "SN74LVC1G08DCKR" H 5844 4447 60  0000 L CNN
 F 2 "digikey-footprints:SC-70-5" H 5700 4700 60  0001 L CNN
@@
 AR Path="/5EF588A2/5EFA444C" Ref="R303"  Part="1"
 AR Path="/5EFCF919/5EFA444C" Ref="R203"  Part="1"
-F 0 "R203" H 3120 3946 50  0000 L CNN
+F 0 "R303" H 3120 3946 50  0000 L CNN
 F 1 "100k" H 3120 3855 50  0000 L CNN
 F 2 "" V 2980 3900 50  0001 C CNN
@@
 AR Path="/5EF588A2/5EFA4E4F" Ref="#PWR0110"  Part="1"
 AR Path="/5EFCF919/5EFA4E4F" Ref="#PWR0118"  Part="1"
-F 0 "#PWR0118" H 3050 4050 50  0001 C CNN
+F 0 "#PWR0110" H 3050 4050 50  0001 C CNN
 F 1 "GND" H 3055 4127 50  0000 C CNN
 F 2 "" H 3050 4300 50  0001 C CNN
@@
 AR Path="/5EF588A2/5EFA6D3C" Ref="#PWR0111"  Part="1"
 AR Path="/5EFCF919/5EFA6D3C" Ref="#PWR0119"  Part="1"
-F 0 "#PWR0119" H 5500 4750 50  0001 C CNN
+F 0 "#PWR0111" H 5500 4750 50  0001 C CNN
 F 1 "GND" H 5505 4827 50  0000 C CNN
 F 2 "" H 5500 5000 50  0001 C CNN
@@
 Wire Wire Line
 	5500 5000 5500 4800
-Text HLabel 2800 4800 0    50   Input ~ 0
-ErrSig1
-Wire Wire Line
-	2800 4800 3400 4800
-Wire Wire Line
-	3400 4800 3400 4600
 Wire Wire Line
 	7150 4450 5850 4450
@@
 L 2020-06-28_23-59-59:SN74LVC1G14DCKR U301
 U 1 1 5EFB2E9F
-P 3200 5700
+P 1700 5100
 AR Path="/5EF588A2/5EFB2E9F" Ref="U301"  Part="1"
 AR Path="/5EFCF919/5EFB2E9F" Ref="U201"  Part="1"
-F 0 "U201" H 4300 6087 60  0000 C CNN
-F 1 "SN74LVC1G14DCKR" H 4300 5981 60  0000 C CNN
-F 2 "DCK5" H 4300 5940 60  0001 C CNN
-F 3 "" H 3200 5700 60  0000 C CNN
-	1    3200 5700
+F 0 "U301" H 2800 5487 60  0000 C CNN
+F 1 "SN74LVC1G14DCKR" H 2800 5381 60  0000 C CNN
+F 2 "DCK5" H 2800 5340 60  0001 C CNN
+F 3 "" H 1700 5100 60  0000 C CNN
+	1    1700 5100
 	1    0    0    -1
 $EndComp
@@
 L power:GND #PWR0112
 U 1 1 5EFB4DC8
-P 5700 5900
+P 4200 5300
 AR Path="/5EF588A2/5EFB4DC8" Ref="#PWR0112"  Part="1"
 AR Path="/5EFCF919/5EFB4DC8" Ref="#PWR0120"  Part="1"
-F 0 "#PWR0120" H 5700 5650 50  0001 C CNN
-F 1 "GND" H 5705 5727 50  0000 C CNN
-F 2 "" H 5700 5900 50  0001 C CNN
-F 3 "" H 5700 5900 50  0001 C CNN
-	1    5700 5900
-	1    0    0    -1
-$EndComp
-Wire Wire Line
-	5700 5900 5400 5900
-NoConn ~ 3200 5700
-Wire Wire Line
-	3800 4600 3800 5100
-Wire Wire Line
-	3800 5100 3000 5100
-Wire Wire Line
-	3000 5100 3000 5800
-Wire Wire Line
-	3000 5800 3200 5800
-Wire Wire Line
-	3400 4600 3800 4600
-Wire Wire Line
-	4700 5300 4700 4600
-Wire Wire Line
-	4700 4600 5200 4600
+F 0 "#PWR0112" H 4200 5050 50  0001 C CNN
+F 1 "GND" H 4205 5127 50  0000 C CNN
+F 2 "" H 4200 5300 50  0001 C CNN
+F 3 "" H 4200 5300 50  0001 C CNN
+	1    4200 5300
+	1    0    0    -1
+$EndComp
+Wire Wire Line
+	4200 5300 3900 5300
+NoConn ~ 1700 5100
 Wire Wire Line
 	3300 4400 5200 4400
 Wire Wire Line
-	5400 5800 5500 5800
-Wire Wire Line
-	5500 5800 5500 5300
-Wire Wire Line
-	4700 5300 5500 5300
+	3900 5200 4000 5200
 $Comp
 L BSS138W:BSS138W Q302
@@
 AR Path="/5EF588A2/5EFB94AA" Ref="Q302"  Part="1"
 AR Path="/5EFCF919/5EFB94AA" Ref="Q202"  Part="1"
-F 0 "Q202" V 7493 4350 50  0000 C CNN
+F 0 "Q302" V 7493 4350 50  0000 C CNN
 F 1 "BSS138W" V 7584 4350 50  0000 C CNN
 F 2 "SOT323-R" H 7350 4350 50  0001 L BNN
@@
 AR Path="/5EF588A2/5EFBA4E9" Ref="#PWR0113"  Part="1"
 AR Path="/5EFCF919/5EFBA4E9" Ref="#PWR0121"  Part="1"
-F 0 "#PWR0121" H 7350 4500 50  0001 C CNN
+F 0 "#PWR0113" H 7350 4500 50  0001 C CNN
 F 1 "GND" H 7355 4577 50  0000 C CNN
 F 2 "" H 7350 4750 50  0001 C CNN
@@
 AR Path="/5EF588A2/5EFBB268" Ref="D303"  Part="1"
 AR Path="/5EFCF919/5EFBB268" Ref="D203"  Part="1"
-F 0 "D203" H 7300 3653 60  0000 C CNN
+F 0 "D303" H 7300 3653 60  0000 C CNN
 F 1 "LTST-C150KRKT" H 7300 3759 60  0000 C CNN
 F 2 "digikey-footprints:1206" H 7550 4100 60  0001 L CNN
@@
 AR Path="/5EF588A2/5EFBC18E" Ref="R304"  Part="1"
 AR Path="/5EFCF919/5EFBC18E" Ref="R204"  Part="1"
-F 0 "R204" H 7420 3396 50  0000 L CNN
-F 1 "500" H 7420 3305 50  0000 L CNN
+F 0 "R304" H 7420 3396 50  0000 L CNN
+F 1 "1k" H 7420 3305 50  0000 L CNN
 F 2 "" V 7280 3350 50  0001 C CNN
 F 3 "~" H 7350 3350 50  0001 C CNN
@@
 +5Vin
 Wire Wire Line
-	5500 3900 5500 4200
-Text HLabel 6000 5700 2    50   Input ~ 0
-+5Vin
-Wire Wire Line
-	5400 5700 6000 5700
+	5500 3900 5500 4050
+Text HLabel 4500 5100 2    50   Input ~ 0
++5Vin
+Wire Wire Line
+	3900 5100 4500 5100
+Wire Wire Line
+	1500 5200 1700 5200
+Text HLabel 1500 5200 0    50   Input ~ 0
+ErrSig1
+Wire Wire Line
+	4000 4600 5200 4600
+Wire Wire Line
+	4000 4600 4000 5200
+$Comp
+L Device:C C301
+U 1 1 5F0541C1
+P 5650 4050
+AR Path="/5EF588A2/5F0541C1" Ref="C301"  Part="1"
+AR Path="/5EFCF919/5F0541C1" Ref="C201"  Part="1"
+F 0 "C301" V 5398 4050 50  0000 C CNN
+F 1 "0.1u" V 5489 4050 50  0000 C CNN
+F 2 "" H 5688 3900 50  0001 C CNN
+F 3 "~" H 5650 4050 50  0001 C CNN
+	1    5650 4050
+	0    1    1    0
+$EndComp
+Connection ~ 5500 4050
+Wire Wire Line
+	5500 4050 5500 4200
+$Comp
+L power:GND #PWR0301
+U 1 1 5F0549D4
+P 6050 4050
+AR Path="/5EF588A2/5F0549D4" Ref="#PWR0301"  Part="1"
+AR Path="/5EFCF919/5F0549D4" Ref="#PWR0201"  Part="1"
+F 0 "#PWR0301" H 6050 3800 50  0001 C CNN
+F 1 "GND" H 6055 3877 50  0000 C CNN
+F 2 "" H 6050 4050 50  0001 C CNN
+F 3 "" H 6050 4050 50  0001 C CNN
+	1    6050 4050
+	1    0    0    -1
+$EndComp
+Wire Wire Line
+	6050 4050 5800 4050
 $EndSCHEMATC
