File: relay_interlock.sch (KiCad schematic (older format))
At the start: 14 parts, among them Q301 BSS138W, Q302 BSS138W, SW301 SW_Push, U301 SN74LVC1G14DCKR, U302 SR4D4005, U303 SN74LVC1G08DCKR

Commit message: Adding Footprints
Parts:
- C301: footprint (none) -> Capacitor_SMD:C_1206_3216Metric_Pad1.42x1.75mm_HandSolder
- D301, D302, D303: footprint digikey-footprints:1206 -> LED_SMD:LED_1206_3216Metric_Pad1.42x1.75mm_HandSolder
- Q301, Q302: footprint SOT323-R -> BSS138W:SOT323-R
- R301, R302, R303, R304: footprint (none) -> Resistor_SMD:R_1206_3216Metric_Pad1.42x1.75mm_HandSolder
- U301: footprint DCK5 -> inverter:SN74LVC1G14DCKR
- U302: footprint RELAY10-5MM-6.5MM -> SRD4005:SR4D4005
- U303: footprint digikey-footprints:SC-70-5 -> inverter:SN74LVC1G14DCKR
Changed lines of the file:
@@
 F 0 "Q301" V 6443 2650 50  0000 C CNN
 F 1 "BSS138W" V 6534 2650 50  0000 C CNN
-F 2 "SOT323-R" H 6300 2650 50  0001 L BNN
+F 2 "BSS138W:SOT323-R" H 6300 2650 50  0001 L BNN
 F 3 "" H 6300 2650 50  0001 C CNN
 	1    6300 2650
@@
 F 0 "U302" H 4900 3138 60  0000 C CNN
 F 1 "SR4D4005" H 4900 3032 60  0000 C CNN
-F 2 "RELAY10-5MM-6.5MM" H 4900 2990 60  0001 C CNN
+F 2 "SRD4005:SR4D4005" H 4900 2990 60  0001 C CNN
 F 3 "" H 4000 2650 60  0000 C CNN
 	1    4000 2650
@@
 F 0 "D301" H 2150 2753 60  0000 C CNN
 F 1 "LTST-C150KRKT" H 2150 2859 60  0000 C CNN
-F 2 "digikey-footprints:1206" H 2400 3200 60  0001 L CNN
+F 2 "LED_SMD:LED_1206_3216Metric_Pad1.42x1.75mm_HandSolder" H 2400 3200 60  0001 L CNN
 F 3 "http://optoelectronics.liteon.com/upload/download/DS-22-99-0149/LTST-C150KRKT.pdf" H 2400 3300 60  0001 L CNN
 F 4 "160-1405-1-ND" H 2400 3400 60  0001 L CNN "Digi-Key_PN"
@@
 F 0 "R301" H 1870 3196 50  0000 L CNN
 F 1 "1k" H 1870 3105 50  0000 L CNN
-F 2 "" V 1730 3150 50  0001 C CNN
+F 2 "Resistor_SMD:R_1206_3216Metric_Pad1.42x1.75mm_HandSolder" V 1730 3150 50  0001 C CNN
 F 3 "~" H 1800 3150 50  0001 C CNN
 	1    1800 3150
@@
 F 0 "D302" H 2550 3203 60  0000 C CNN
 F 1 "LTST-C150KGKT" H 2550 3309 60  0000 C CNN
-F 2 "digikey-footprints:1206" H 2800 3650 60  0001 L CNN
+F 2 "LED_SMD:LED_1206_3216Metric_Pad1.42x1.75mm_HandSolder" H 2800 3650 60  0001 L CNN
 F 3 "http://optoelectronics.liteon.com/upload/download/DS22-2000-072/LTST-C150KGKT.pdf" H 2800 3750 60  0001 L CNN
 F 4 "160-1404-1-ND" H 2800 3850 60  0001 L CNN "Digi-Key_PN"
@@
 F 0 "R302" H 2570 3896 50  0000 L CNN
 F 1 "1k" H 2570 3805 50  0000 L CNN
-F 2 "" V 2430 3850 50  0001 C CNN
+F 2 "Resistor_SMD:R_1206_3216Metric_Pad1.42x1.75mm_HandSolder" V 2430 3850 50  0001 C CNN
 F 3 "~" H 2500 3850 50  0001 C CNN
 	1    2500 3850
@@
 F 0 "U303" H 5844 4553 60  0000 L CNN
 F 1 "SN74LVC1G08DCKR" H 5844 4447 60  0000 L CNN
-F 2 "digikey-footprints:SC-70-5" H 5700 4700 60  0001 L CNN
+F 2 "inverter:SN74LVC1G14DCKR" H 5700 4700 60  0001 L CNN
 F 3 "http://www.ti.com/general/docs/suppproductinfo.tsp?distId=10&gotoUrl=http%3A%2F%2Fwww.ti.com%2Flit%2Fgpn%2Fsn74lvc1g08" H 5700 4800 60  0001 L CNN
 F 4 "296-11602-1-ND" H 5700 4900 60  0001 L CNN "Digi-Key_PN"
@@
 F 0 "R303" H 3120 3946 50  0000 L CNN
 F 1 "100k" H 3120 3855 50  0000 L CNN
-F 2 "" V 2980 3900 50  0001 C CNN
+F 2 "Resistor_SMD:R_1206_3216Metric_Pad1.42x1.75mm_HandSolder" V 2980 3900 50  0001 C CNN
 F 3 "~" H 3050 3900 50  0001 C CNN
 	1    3050 3900
@@
 F 0 "U301" H 2800 5487 60  0000 C CNN
 F 1 "SN74LVC1G14DCKR" H 2800 5381 60  0000 C CNN
-F 2 "DCK5" H 2800 5340 60  0001 C CNN
+F 2 "inverter:SN74LVC1G14DCKR" H 2800 5340 60  0001 C CNN
 F 3 "" H 1700 5100 60  0000 C CNN
 	1    1700 5100
@@
 F 0 "Q302" V 7493 4350 50  0000 C CNN
 F 1 "BSS138W" V 7584 4350 50  0000 C CNN
-F 2 "SOT323-R" H 7350 4350 50  0001 L BNN
+F 2 "BSS138W:SOT323-R" H 7350 4350 50  0001 L BNN
 F 3 "" H 7350 4350 50  0001 C CNN
 	1    7350 4350
@@
 F 0 "D303" H 7300 3653 60  0000 C CNN
 F 1 "LTST-C150KRKT" H 7300 3759 60  0000 C CNN
-F 2 "digikey-footprints:1206" H 7550 4100 60  0001 L CNN
+F 2 "LED_SMD:LED_1206_3216Metric_Pad1.42x1.75mm_HandSolder" H 7550 4100 60  0001 L CNN
 F 3 "http://optoelectronics.liteon.com/upload/download/DS-22-99-0149/LTST-C150KRKT.pdf" H 7550 4200 60  0001 L CNN
 F 4 "160-1405-1-ND" H 7550 4300 60  0001 L CNN "Digi-Key_PN"
@@
 F 0 "R304" H 7420 3396 50  0000 L CNN
 F 1 "1k" H 7420 3305 50  0000 L CNN
-F 2 "" V 7280 3350 50  0001 C CNN
+F 2 "Resistor_SMD:R_1206_3216Metric_Pad1.42x1.75mm_HandSolder" V 7280 3350 50  0001 C CNN
 F 3 "~" H 7350 3350 50  0001 C CNN
 	1    7350 3350
@@
 F 0 "C301" V 5398 4050 50  0000 C CNN
 F 1 "0.1u" V 5489 4050 50  0000 C CNN
-F 2 "" H 5688 3900 50  0001 C CNN
+F 2 "Capacitor_SMD:C_1206_3216Metric_Pad1.42x1.75mm_HandSolder" H 5688 3900 50  0001 C CNN
 F 3 "~" H 5650 4050 50  0001 C CNN
 	1    5650 4050

Commit message: All Footprints assembled!
Parts:
- SW301: footprint (none) -> Magnet_PS_Interlock:TP11SH8CQE
Changed lines of the file:
@@
 $Descr A4 11693 8268
 encoding utf-8
-Sheet 3 3
+Sheet 2 3
 Title ""
 Date ""
@@
 AR Path="/5EF588A2/5EF5F5C0" Ref="SW301"  Part="1"
 AR Path="/5EFCF919/5EF5F5C0" Ref="SW201"  Part="1"
-F 0 "SW301" H 3200 2935 50  0000 C CNN
+F 0 "SW201" H 3200 2935 50  0000 C CNN
 F 1 "SW_Push" H 3200 2844 50  0000 C CNN
-F 2 "" H 3200 2850 50  0001 C CNN
+F 2 "Magnet_PS_Interlock:TP11SH8CQE" H 3200 2850 50  0001 C CNN
 F 3 "~" H 3200 2850 50  0001 C CNN
 	1    3200 2650
@@
 AR Path="/5EF588A2/5EFBAF07" Ref="Q301"  Part="1"
 AR Path="/5EFCF919/5EFBAF07" Ref="Q201"  Part="1"
-F 0 "Q301" V 6443 2650 50  0000 C CNN
+F 0 "Q201" V 6443 2650 50  0000 C CNN
 F 1 "BSS138W" V 6534 2650 50  0000 C CNN
 F 2 "BSS138W:SOT323-R" H 6300 2650 50  0001 L BNN
@@
 AR Path="/5EF588A2/5EFC1523" Ref="#PWR0107"  Part="1"
 AR Path="/5EFCF919/5EFC1523" Ref="#PWR0115"  Part="1"
-F 0 "#PWR0107" H 6700 2400 50  0001 C CNN
+F 0 "#PWR0115" H 6700 2400 50  0001 C CNN
 F 1 "GND" H 6705 2477 50  0000 C CNN
 F 2 "" H 6700 2650 50  0001 C CNN
@@
 AR Path="/5EF588A2/5EFBABE7" Ref="U302"  Part="1"
 AR Path="/5EFCF919/5EFBABE7" Ref="U202"  Part="1"
-F 0 "U302" H 4900 3138 60  0000 C CNN
+F 0 "U202" H 4900 3138 60  0000 C CNN
 F 1 "SR4D4005" H 4900 3032 60  0000 C CNN
 F 2 "SRD4005:SR4D4005" H 4900 2990 60  0001 C CNN
@@
 AR Path="/5EF588A2/5EFD24D7" Ref="D301"  Part="1"
 AR Path="/5EFCF919/5EFD24D7" Ref="D201"  Part="1"
-F 0 "D301" H 2150 2753 60  0000 C CNN
+F 0 "D201" H 2150 2753 60  0000 C CNN
 F 1 "LTST-C150KRKT" H 2150 2859 60  0000 C CNN
 F 2 "LED_SMD:LED_1206_3216Metric_Pad1.42x1.75mm_HandSolder" H 2400 3200 60  0001 L CNN
@@
 AR Path="/5EF588A2/5EFD53B2" Ref="R301"  Part="1"
 AR Path="/5EFCF919/5EFD53B2" Ref="R201"  Part="1"
-F 0 "R301" H 1870 3196 50  0000 L CNN
+F 0 "R201" H 1870 3196 50  0000 L CNN
 F 1 "1k" H 1870 3105 50  0000 L CNN
 F 2 "Resistor_SMD:R_1206_3216Metric_Pad1.42x1.75mm_HandSolder" V 1730 3150 50  0001 C CNN
@@
 AR Path="/5EF588A2/5EFD6108" Ref="#PWR0108"  Part="1"
 AR Path="/5EFCF919/5EFD6108" Ref="#PWR0116"  Part="1"
-F 0 "#PWR0108" H 1800 3300 50  0001 C CNN
+F 0 "#PWR0116" H 1800 3300 50  0001 C CNN
 F 1 "GND" H 1805 3377 50  0000 C CNN
 F 2 "" H 1800 3550 50  0001 C CNN
@@
 AR Path="/5EF588A2/5EFD7D41" Ref="D302"  Part="1"
 AR Path="/5EFCF919/5EFD7D41" Ref="D202"  Part="1"
-F 0 "D302" H 2550 3203 60  0000 C CNN
+F 0 "D202" H 2550 3203 60  0000 C CNN
 F 1 "LTST-C150KGKT" H 2550 3309 60  0000 C CNN
 F 2 "LED_SMD:LED_1206_3216Metric_Pad1.42x1.75mm_HandSolder" H 2800 3650 60  0001 L CNN
@@
 AR Path="/5EF588A2/5EFDCB0F" Ref="R302"  Part="1"
 AR Path="/5EFCF919/5EFDCB0F" Ref="R202"  Part="1"
-F 0 "R302" H 2570 3896 50  0000 L CNN
+F 0 "R202" H 2570 3896 50  0000 L CNN
 F 1 "1k" H 2570 3805 50  0000 L CNN
 F 2 "Resistor_SMD:R_1206_3216Metric_Pad1.42x1.75mm_HandSolder" V 2430 3850 50  0001 C CNN
@@
 AR Path="/5EF588A2/5EFDD582" Ref="#PWR0109"  Part="1"
 AR Path="/5EFCF919/5EFDD582" Ref="#PWR0117"  Part="1"
-F 0 "#PWR0109" H 2500 3950 50  0001 C CNN
+F 0 "#PWR0117" H 2500 3950 50  0001 C CNN
 F 1 "GND" H 2505 4027 50  0000 C CNN
 F 2 "" H 2500 4200 50  0001 C CNN
@@
 AR Path="/5EF588A2/5EF92FF9" Ref="U303"  Part="1"
 AR Path="/5EFCF919/5EF92FF9" Ref="U203"  Part="1"
-F 0 "U303" H 5844 4553 60  0000 L CNN
+F 0 "U203" H 5844 4553 60  0000 L CNN
 F 1 "SN74LVC1G08DCKR" H 5844 4447 60  0000 L CNN
 F 2 "inverter:SN74LVC1G14DCKR" H 5700 4700 60  0001 L CNN
@@
 AR Path="/5EF588A2/5EFA444C" Ref="R303"  Part="1"
 AR Path="/5EFCF919/5EFA444C" Ref="R203"  Part="1"
-F 0 "R303" H 3120 3946 50  0000 L CNN
+F 0 "R203" H 3120 3946 50  0000 L CNN
 F 1 "100k" H 3120 3855 50  0000 L CNN
 F 2 "Resistor_SMD:R_1206_3216Metric_Pad1.42x1.75mm_HandSolder" V 2980 3900 50  0001 C CNN
@@
 AR Path="/5EF588A2/5EFA4E4F" Ref="#PWR0110"  Part="1"
 AR Path="/5EFCF919/5EFA4E4F" Ref="#PWR0118"  Part="1"
-F 0 "#PWR0110" H 3050 4050 50  0001 C CNN
+F 0 "#PWR0118" H 3050 4050 50  0001 C CNN
 F 1 "GND" H 3055 4127 50  0000 C CNN
 F 2 "" H 3050 4300 50  0001 C CNN
@@
 AR Path="/5EF588A2/5EFA6D3C" Ref="#PWR0111"  Part="1"
 AR Path="/5EFCF919/5EFA6D3C" Ref="#PWR0119"  Part="1"
-F 0 "#PWR0111" H 5500 4750 50  0001 C CNN
+F 0 "#PWR0119" H 5500 4750 50  0001 C CNN
 F 1 "GND" H 5505 4827 50  0000 C CNN
 F 2 "" H 5500 5000 50  0001 C CNN
@@
 AR Path="/5EF588A2/5EFB2E9F" Ref="U301"  Part="1"
 AR Path="/5EFCF919/5EFB2E9F" Ref="U201"  Part="1"
-F 0 "U301" H 2800 5487 60  0000 C CNN
+F 0 "U201" H 2800 5487 60  0000 C CNN
 F 1 "SN74LVC1G14DCKR" H 2800 5381 60  0000 C CNN
 F 2 "inverter:SN74LVC1G14DCKR" H 2800 5340 60  0001 C CNN
@@
 AR Path="/5EF588A2/5EFB4DC8" Ref="#PWR0112"  Part="1"
 AR Path="/5EFCF919/5EFB4DC8" Ref="#PWR0120"  Part="1"
-F 0 "#PWR0112" H 4200 5050 50  0001 C CNN
+F 0 "#PWR0120" H 4200 5050 50  0001 C CNN
 F 1 "GND" H 4205 5127 50  0000 C CNN
 F 2 "" H 4200 5300 50  0001 C CNN
@@
 AR Path="/5EF588A2/5EFB94AA" Ref="Q302"  Part="1"
 AR Path="/5EFCF919/5EFB94AA" Ref="Q202"  Part="1"
-F 0 "Q302" V 7493 4350 50  0000 C CNN
+F 0 "Q202" V 7493 4350 50  0000 C CNN
 F 1 "BSS138W" V 7584 4350 50  0000 C CNN
 F 2 "BSS138W:SOT323-R" H 7350 4350 50  0001 L BNN
@@
 AR Path="/5EF588A2/5EFBA4E9" Ref="#PWR0113"  Part="1"
 AR Path="/5EFCF919/5EFBA4E9" Ref="#PWR0121"  Part="1"
-F 0 "#PWR0113" H 7350 4500 50  0001 C CNN
+F 0 "#PWR0121" H 7350 4500 50  0001 C CNN
 F 1 "GND" H 7355 4577 50  0000 C CNN
 F 2 "" H 7350 4750 50  0001 C CNN
@@
 AR Path="/5EF588A2/5EFBB268" Ref="D303"  Part="1"
 AR Path="/5EFCF919/5EFBB268" Ref="D203"  Part="1"
-F 0 "D303" H 7300 3653 60  0000 C CNN
+F 0 "D203" H 7300 3653 60  0000 C CNN
 F 1 "LTST-C150KRKT" H 7300 3759 60  0000 C CNN
 F 2 "LED_SMD:LED_1206_3216Metric_Pad1.42x1.75mm_HandSolder" H 7550 4100 60  0001 L CNN
@@
 AR Path="/5EF588A2/5EFBC18E" Ref="R304"  Part="1"
 AR Path="/5EFCF919/5EFBC18E" Ref="R204"  Part="1"
-F 0 "R304" H 7420 3396 50  0000 L CNN
+F 0 "R204" H 7420 3396 50  0000 L CNN
 F 1 "1k" H 7420 3305 50  0000 L CNN
 F 2 "Resistor_SMD:R_1206_3216Metric_Pad1.42x1.75mm_HandSolder" V 7280 3350 50  0001 C CNN
@@
 AR Path="/5EF588A2/5F0541C1" Ref="C301"  Part="1"
 AR Path="/5EFCF919/5F0541C1" Ref="C201"  Part="1"
-F 0 "C301" V 5398 4050 50  0000 C CNN
+F 0 "C201" V 5398 4050 50  0000 C CNN
 F 1 "0.1u" V 5489 4050 50  0000 C CNN
 F 2 "Capacitor_SMD:C_1206_3216Metric_Pad1.42x1.75mm_HandSolder" H 5688 3900 50  0001 C CNN
@@
 AR Path="/5EF588A2/5F0549D4" Ref="#PWR0301"  Part="1"
 AR Path="/5EFCF919/5F0549D4" Ref="#PWR0201"  Part="1"
-F 0 "#PWR0301" H 6050 3800 50  0001 C CNN
+F 0 "#PWR0201" H 6050 3800 50  0001 C CNN
 F 1 "GND" H 6055 3877 50  0000 C CNN
 F 2 "" H 6050 4050 50  0001 C CNN
