File: magnets_interlock.kicad_pcb (KiCad board)
At the start: 2 copper layers, 114.3 x 72.4 mm, 47 parts, among them Q201 BSS138W, Q202 BSS138W, Q301 BSS138W, Q302 BSS138W, SW201 SW_Push, SW301 SW_Push, U101 Si8640BD-B-IS, U201 SN74LVC1G14DCKR, U202 SR4D4005, U203 SN74LVC1G08DCKR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

Commit message: Enrique changes
Parts:
- removed C101: 4.7u, Capacitor_SMD:C_1206_3216Metric_Pad1.42x1.75mm_HandSolder
- removed C102: 2.2u, Capacitor_SMD:C_1206_3216Metric_Pad1.42x1.75mm_HandSolder
- removed VT101: NXJ1S0505MC-R7, NXJ1S050:VREG_NXJ1S0505MC-R7
- added C109: 47u, Capacitor_THT:CP_Radial_D8.0mm_P3.50mm, F.Cu at (227.6, 54.4)
- added C110: 4.7u, Capacitor_SMD:C_1206_3216Metric_Pad1.42x1.75mm_HandSolder, F.Cu at (216.1, 49.5)
- added C111: 4.7u, Capacitor_SMD:C_1206_3216Metric_Pad1.42x1.75mm_HandSolder, F.Cu at (215.7, 52.1)
- U303: value SN74LVC1G08 -> SN74LVC1G08DCKR
- moved C104 31.2 mm to (197.9, 68.6), turned to 180 degrees
- moved VT102 21.2 mm to (197.7, 61.0), turned to 0 degrees
- moved C108 19.1 mm to (197.9, 53.3)
- moved C103 12.8 mm to (158.8, 68.6), turned to 180 degrees
- moved VT103 2.19 mm to (159.6, 61.0), turned to 0 degrees
- moved SW201 1.27 mm to (157.5, 73.7)
Connections:
- C105 pad 1: Net-(C102-Pad1) -> +5VIN
- C105 pad 2: Net-(C102-Pad2) -> PWR_GND_IN
- ERR_In101 pad 2: Net-(C102-Pad2) -> PWR_GND_IN
- ERR_In101 pad 3: Net-(C102-Pad2) -> PWR_GND_IN
- ERR_In101 pad 4: Net-(C102-Pad2) -> PWR_GND_IN
- U101 pad 1: Net-(C102-Pad1) -> +5VIN
- U101 pad 2: Net-(C102-Pad2) -> PWR_GND_IN
- U101 pad 5: Net-(C102-Pad2) -> PWR_GND_IN
- U101 pad 6: Net-(C102-Pad2) -> PWR_GND_IN
- U101 pad 8: Net-(C102-Pad2) -> PWR_GND_IN
Other:
- board size 114.3 x 72.4 mm -> 119.4 x 72.4 mm

Commit message: Draft 1 Almost There
Parts:
- removed C108: 4.7u, Capacitor_SMD:C_1206_3216Metric_Pad1.42x1.75mm_HandSolder
- removed MAG_ENABLE_OUT101: BNC_Input_female, BNC_female:1-1337543-0
- removed VT103: NXJ1S0505MC-R7, NXJ1S050:VREG_NXJ1S0505MC-R7
- added C101: 0.1u, Capacitor_SMD:C_1206_3216Metric_Pad1.42x1.75mm_HandSolder, F.Cu at (245.7, 59.6)
- added C102: 2.2u, Capacitor_SMD:C_1206_3216Metric_Pad1.42x1.75mm_HandSolder, F.Cu at (199.1, 70.6)
- added D204: D_TVS_ALT, TVS diode:SM15T15CA, F.Cu at (269.7, 73.0)
- added D304: D_TVS_ALT, TVS diode:SM15T15CA, F.Cu at (269.7, 61.9)
- added L101: 4.7u, VLCF4024T-4R7N1R4-2:VLCF4024T-4R7N1R4-2, F.Cu at (193.0, 51.8)
- added L102: 10u, VLCF4024T-4R7N1R4-2:VLCF4024T-4R7N1R4-2, F.Cu at (203.2, 70.8)
- added L103: 4.7u, VLCF4024T-4R7N1R4-2:VLCF4024T-4R7N1R4-2, F.Cu at (154.4, 51.8)
- added L104: 10u, VLCF4024T-4R7N1R4-2:VLCF4024T-4R7N1R4-2, F.Cu at (164.6, 70.6)
- added Relay_Off_Output101: BNC_Input_female, BNC_female:1-1337543-0, F.Cu at (234.9, 90.2)
- added S102: CL-SB-12B-01T, CL-SB-12B-01T:CL-SB-12B, F.Cu at (208.5, 85.4)
- added U102: SN74LVC1G08DCKR, inverter:SN74LVC1G14DCKR, F.Cu at (218.8, 89.4)
- added U103: 691321100003, Magnet_PS_Interlock:691321100003, F.Cu at (243.8, 109.2)
- added VT101: NXJ1S0505MC-R7, NXJ1S050:VREG_NXJ1S0505MC-R7, F.Cu at (159.8, 61.2)
- C103: value 2.2u -> 4.7u
- R102, R103: value 1k -> 10k
- U101: value Si8640BD-B-IS -> DW0016B_N_TEX; footprint SI8640DBIS:Si8640BD-B-IS -> ISO7741FDWR:ISO7741FDWR
- moved C104 39.2 mm to (158.8, 69.3)
- moved C107 37.3 mm to (197.1, 51.6), turned to 270 degrees
- moved C105 27.4 mm to (207.8, 74.9), turned to 180 degrees
- moved C103 16.7 mm to (159.0, 51.9), turned to 270 degrees
- moved R102 11.9 mm to (227.5, 78.7), turned to 180 degrees
- moved R103 10.5 mm to (213.1, 91.4)
- moved C106 10.1 mm to (226.6, 74.4), turned to 180 degrees
- moved U101 9.82 mm to (216.7, 78.2), turned to 0 degrees
- moved SW301 2.70 mm to (196.3, 75.7), turned to 180 degrees
- moved C109 2.55 mm to (227.8, 51.8), turned to 270 degrees
- moved SW201 0.57 mm to (157.7, 74.2)
Connections:
- C103 pad 1: +5VOut2 -> +5VIN
- C103 pad 2: GND -> PWR_GND_IN
- C104 pad 1: +5VOut1 -> +5VOut2
- C109 pad 1: PWR_GND_IN -> +5VIN
- C109 pad 2: +5VIN -> PWR_GND_IN
- D202 pad 1: Net-(D202-Pad1) -> /Relay_2/Relay-Off-Sig
- D302 pad 1: Net-(D302-Pad1) -> /Relay_1/Relay-Off-Sig
- Q201 pad 2: Net-(Q201-Pad2) -> GND
- Q201 pad 3: GND -> Net-(Q201-Pad3)
- Q301 pad 2: Net-(Q301-Pad2) -> GND
- Q301 pad 3: GND -> Net-(Q301-Pad3)
- R103 pad 1: GND -> PWR_GND_IN
- R203 pad 1: Net-(D202-Pad1) -> /Relay_2/Relay-Off-Sig
- R303 pad 1: Net-(D302-Pad1) -> /Relay_1/Relay-Off-Sig
- SW201 pad 2: Net-(D202-Pad1) -> /Relay_2/Relay-Off-Sig
- SW301 pad 2: Net-(D302-Pad1) -> /Relay_1/Relay-Off-Sig
- U101 pad 11: Net-(R103-Pad2) -> Relay_off_signal
- U101 pad 6: PWR_GND_IN -> Net-(Relay_Off_Output101-Pad1)
- U101 pad 7: Net-(U101-Pad7) -> Net-(R103-Pad2)
- U202 pad 11: +5VOut2 -> Net-(U202-Pad11)
- U202 pad 12: Net-(D201-Pad1) -> Net-(U202-Pad12)
- U202 pad 21: Net-(U202-Pad21) -> +5VOut2
- U202 pad 22: Net-(U202-Pad22) -> Net-(D201-Pad1)
- U202 pad 33: +5VOut2 -> /Relay_2/Enable_Conn_2
- U202 pad 34: Net-(D202-Pad1) -> /Relay_2/Enable_Conn_1
- U202 pad 43: /Relay_2/Enable_Conn_2 -> +5VOut2
- U202 pad 44: /Relay_2/Enable_Conn_1 -> /Relay_2/Relay-Off-Sig
- U202 pad A1: Net-(D202-Pad1) -> /Relay_2/Relay-Off-Sig
- U202 pad A2: Net-(Q201-Pad2) -> Net-(Q201-Pad3)
- U203 pad 1: Net-(D202-Pad1) -> /Relay_2/Relay-Off-Sig
- U302 pad 11: +5VOut1 -> Net-(U302-Pad11)
- U302 pad 12: Net-(D301-Pad1) -> Net-(U302-Pad12)
- U302 pad 21: Net-(U302-Pad21) -> +5VOut1
- U302 pad 22: Net-(U302-Pad22) -> Net-(D301-Pad1)
- U302 pad 33: +5VOut1 -> /Relay_2/Enable_Conn_1
- U302 pad 34: Net-(D302-Pad1) -> /Relay_1/Enable_Conn_1
- U302 pad 43: /Relay_2/Enable_Conn_1 -> +5VOut1
- U302 pad 44: /Relay_1/Enable_Conn_1 -> /Relay_1/Relay-Off-Sig
- U302 pad A1: Net-(D302-Pad1) -> /Relay_1/Relay-Off-Sig
- U302 pad A2: Net-(Q301-Pad2) -> Net-(Q301-Pad3)
- U303 pad 1: Net-(D302-Pad1) -> /Relay_1/Relay-Off-Sig
- VT102 pad 3: +5VIN -> Net-(L101-Pad1)
- VT102 pad 8: +5VOut1 -> Net-(L102-Pad2)

Commit message: Next Draft
Parts:
- removed PWR_In101: 691508110303, 3PinPowerTerm:691508110303
- added U104: 691321100003, Magnet_PS_Interlock:691321100003, F.Cu at (215.1, 58.9)
- U101: value DW0016B_N_TEX -> ISO7741FDWR
- moved D204 101.5 mm to (168.9, 84.9), turned to 270 degrees
- moved D304 64.6 mm to (209.6, 85.6), turned to 270 degrees
- moved C101 38.7 mm to (229.4, 94.7), turned to 90 degrees
- moved C106 11.5 mm to (238.0, 73.7)
- moved R102 11.5 mm to (239.0, 78.0)
- moved S101 11.2 mm to (225.8, 68.3)
- moved S102 9.68 mm to (218.2, 86.1)
- moved U102 9.68 mm to (228.4, 90.2)
- moved C105 9.68 mm to (217.5, 75.7)
- moved R101 9.68 mm to (219.2, 70.4)
- moved R103 9.68 mm to (222.8, 92.2)
- moved U101 9.68 mm to (226.3, 78.9)
- moved C109 2.29 mm to (225.6, 51.8)
- moved C102 1.42 mm to (197.8, 71.1), turned to 180 degrees
- moved Q302 1.16 mm to (177.4, 91.9)
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Other:
- board size 119.4 x 72.4 mm -> 120.7 x 72.4 mm
- net class Default: clearance 0.2 -> 0.254; trace_width 0.25 -> 0.254; via_dia 0.8 -> 0.762; via_drill 0.4 -> 0.381
- rule trace_clearance: 0.2 -> 0.254
- rule trace_min: 0.2 -> 0.1524
- rule via_min_drill: 0.3 -> 0.3302
- rule via_min_size: 0.4 -> 0.6858
- board text added: "+5 V IN"
- board text added: "MAGNETS ENABLE OUTPUT"
