File: magnets_interlock.sch (KiCad schematic (older format))
At the start: 9 parts

Commit message: Annotations
Parts:
- R101: renamed from R?; value R -> 10k
- gave numbers to parts that had none: 6
- renumbered ERR_In to ERR_In101, PWR_In to PWR_In101
Connections:
- net +5VOut1: no longer S101.1
- net +5VOut2: now also S101.1
- net GND: now also J101.3 (shield), J101.4 (shield)
- net Relay_2/ErrSig1: now reaches U101.13 (B2)
- net Relay_1/ErrSig1: now reaches U101.14 (B1)
- net Relay_1/Enable_Conn_1: now reaches J101.1 (Center_Pin)
- net Relay_2/Enable_Conn_2: now reaches J101.2 (BNC_Shield)
Changed lines of the file:
@@
 $Descr A4 11693 8268
 encoding utf-8
-Sheet 1 2
+Sheet 1 3
 Title ""
 Date ""
@@
 Comment4 ""
 $EndDescr
-$Sheet
-S 4350 2950 2650 1250
-U 5EF588A2
-F0 "Relays and Mag Enable" 50
-F1 "relay_interlock.sch" 50
-F2 "ErrSig1" I R 7000 3550 50
-F3 "Enable_Conn_1" I R 7000 3950 50
-F4 "Enable_Conn_2" I R 7000 3200 50
-$EndSheet
-$Comp
-L 2020-06-26_17-59-50:Si8640BD-B-IS U?
+$Comp
+L 2020-06-26_17-59-50:Si8640BD-B-IS U101
 U 1 1 5EF654E5
 P 4050 1100
-F 0 "U?" H 5250 1487 60  0000 C CNN
+F 0 "U101" H 5250 1487 60  0000 C CNN
 F 1 "Si8640BD-B-IS" H 5250 1381 60  0000 C CNN
 F 2 "SOIC-16W_SIL" H 5250 1340 60  0001 C CNN
@@
 $EndComp
 $Comp
-L 691508110303:691508110303 PWR_In
+L 691508110303:691508110303 PWR_In101
 U 1 1 5EF7A439
 P 1000 1500
-F 0 "PWR_In" H 943 1867 50  0000 C CNN
+F 0 "PWR_In101" H 943 1867 50  0000 C CNN
 F 1 "691508110303" H 943 1776 50  0000 C CNN
 F 2 "691508110303" H 1000 1500 50  0001 L BNN
@@
 NoConn ~ 1250 1500
 $Comp
-L NXJ1S0505MC-R7:NXJ1S0505MC-R7 VT?
+L NXJ1S0505MC-R7:NXJ1S0505MC-R7 VT101
 U 1 1 5EF9CB9B
 P 1800 2200
-AR Path="/5EF9CB9B" Ref="VT?"  Part="1"
+AR Path="/5EF9CB9B" Ref="VT101"  Part="1"
 AR Path="/5EF82676/5EF9CB9B" Ref="VT?"  Part="1"
-F 0 "VT?" H 1800 1925 50  0000 C CNN
+F 0 "VT101" H 1800 1925 50  0000 C CNN
 F 1 "NXJ1S0505MC-R7" H 1800 1834 50  0000 C CNN
 F 2 "VREG_NXJ1S0505MC-R7" H 1350 1800 50  0001 L BNN
@@
 $EndComp
 $Comp
-L NXJ1S0505MC-R7:NXJ1S0505MC-R7 VT?
+L NXJ1S0505MC-R7:NXJ1S0505MC-R7 VT102
 U 1 1 5EF9D3DC
 P 1800 3150
-AR Path="/5EF9D3DC" Ref="VT?"  Part="1"
+AR Path="/5EF9D3DC" Ref="VT102"  Part="1"
 AR Path="/5EF82676/5EF9D3DC" Ref="VT?"  Part="1"
-F 0 "VT?" H 1800 2875 50  0000 C CNN
+F 0 "VT102" H 1800 2875 50  0000 C CNN
 F 1 "NXJ1S0505MC-R7" H 1800 2784 50  0000 C CNN
 F 2 "VREG_NXJ1S0505MC-R7" H 1350 2750 50  0001 L BNN
@@
 $EndComp
 $Comp
-L NXJ1S0505MC-R7:NXJ1S0505MC-R7 VT?
+L NXJ1S0505MC-R7:NXJ1S0505MC-R7 VT103
 U 1 1 5EF9D5EE
 P 1800 4100
-AR Path="/5EF9D5EE" Ref="VT?"  Part="1"
+AR Path="/5EF9D5EE" Ref="VT103"  Part="1"
 AR Path="/5EF82676/5EF9D5EE" Ref="VT?"  Part="1"
-F 0 "VT?" H 1800 3825 50  0000 C CNN
+F 0 "VT103" H 1800 3825 50  0000 C CNN
 F 1 "NXJ1S0505MC-R7" H 1800 3734 50  0000 C CNN
 F 2 "VREG_NXJ1S0505MC-R7" H 1350 3700 50  0001 L BNN
@@
 	1050 4200 1200 4200
 $Comp
-L magnets_interlock_library:BNC_Input_female ERR_In
+L magnets_interlock_library:BNC_Input_female ERR_In101
 U 1 1 5EF9EE1E
 P 3300 1350
-F 0 "ERR_In" H 3542 1637 60  0000 C CNN
+F 0 "ERR_In101" H 3542 1637 60  0000 C CNN
 F 1 "BNC_Input_female" H 3542 1531 60  0000 C CNN
 F 2 "conn2_1-1337543-0_TEC" H 3700 1290 60  0001 C CNN
@@
 	3550 1100 4050 1100
 $Comp
-L CL-SB-12B-01T:CL-SB-12B-01T S?
+L CL-SB-12B-01T:CL-SB-12B-01T S101
 U 1 1 5EFA58AE
 P 7900 1400
-F 0 "S?" H 7900 1127 50  0000 C CNN
+F 0 "S101" H 7900 1127 50  0000 C CNN
 F 1 "CL-SB-12B-01T" H 7900 1036 50  0000 C CNN
 F 2 "CL-SB-12B" H 7900 1400 50  0001 L BNN
@@
 Wire Wire Line
 	8400 1400 8250 1400
-Text GLabel 7450 1400 3    50   Input ~ 0
-+5VOut1
 Wire Wire Line
 	7450 1400 7550 1400
 $Comp
-L Device:R R?
+L Device:R R101
 U 1 1 5EFB1471
 P 7900 850
-F 0 "R?" H 7970 896 50  0000 L CNN
-F 1 "R" H 7970 805 50  0000 L CNN
+F 0 "R101" H 7970 896 50  0000 L CNN
+F 1 "10k" H 7970 805 50  0000 L CNN
 F 2 "" V 7830 850 50  0001 C CNN
 F 3 "~" H 7900 850 50  0001 C CNN
@@
 Connection ~ 7900 1000
 $Comp
-L magnets_interlock_library:BNC_Input_female J?
+L magnets_interlock_library:BNC_Input_female J101
 U 1 1 5EFC2490
 P 8100 3450
-F 0 "J?" H 8628 3353 60  0000 L CNN
+F 0 "J101" H 8628 3353 60  0000 L CNN
 F 1 "BNC_Input_female" H 8628 3247 60  0000 L CNN
 F 2 "conn2_1-1337543-0_TEC" H 8500 3390 60  0001 C CNN
@@
 	1    0    0    -1
 $EndComp
+$Sheet
+S 4300 4650 2750 950
+U 5EFCF919
+F0 "Relay_2" 50
+F1 "relay_interlock.sch" 50
+F2 "ErrSig1" I R 7050 4800 50
+F3 "Enable_Conn_1" I R 7050 5050 50
+F4 "Enable_Conn_2" I R 7050 5300 50
+F5 "+5Vin" I L 4300 5050 50
+$EndSheet
+Text GLabel 4000 3400 0    50   Input ~ 0
++5VOut1
+Wire Wire Line
+	4000 3400 4350 3400
+Text GLabel 3950 5050 0    50   Input ~ 0
++5VOut2
+Wire Wire Line
+	3950 5050 4300 5050
+Wire Wire Line
+	8100 3650 8100 3700
+$Comp
+L power:GND #PWR0114
+U 1 1 5EFD2B4D
+P 7850 3700
+F 0 "#PWR0114" H 7850 3450 50  0001 C CNN
+F 1 "GND" H 7855 3527 50  0000 C CNN
+F 2 "" H 7850 3700 50  0001 C CNN
+F 3 "" H 7850 3700 50  0001 C CNN
+	1    7850 3700
+	1    0    0    -1
+$EndComp
+Wire Wire Line
+	7850 3700 8100 3700
+Connection ~ 8100 3700
+Wire Wire Line
+	8100 3700 8100 3750
+$Sheet
+S 4350 2950 2650 1250
+U 5EF588A2
+F0 "Relay_1" 50
+F1 "relay_interlock.sch" 50
+F2 "ErrSig1" I R 7000 3050 50
+F3 "Enable_Conn_1" I R 7000 3400 50
+F4 "Enable_Conn_2" I R 7000 3800 50
+F5 "+5Vin" I L 4350 3400 50
+$EndSheet
+Wire Wire Line
+	7000 3800 7200 3800
+Wire Wire Line
+	7200 3800 7200 5050
+Wire Wire Line
+	7200 5050 7050 5050
+Wire Wire Line
+	7050 5300 7600 5300
+Wire Wire Line
+	7600 5300 7600 3550
+Wire Wire Line
+	7600 3550 8100 3550
+Wire Wire Line
+	8100 3450 7650 3450
+Wire Wire Line
+	7650 3450 7650 3400
+Wire Wire Line
+	7650 3400 7000 3400
+Wire Wire Line
+	6450 1300 7200 1300
+Wire Wire Line
+	7200 1300 7200 3050
+Wire Wire Line
+	7200 3050 7000 3050
+Wire Wire Line
+	6450 1400 7350 1400
+Wire Wire Line
+	7350 1400 7350 4800
+Wire Wire Line
+	7350 4800 7050 4800
+Text GLabel 7450 1400 3    50   Input ~ 0
++5VOut2
 $EndSCHEMATC

Commit message: Bypass everything and run Error Check
Parts:
- added C101, C107, C108: 4.7u, symbol Device:C
- added C102, C103, C104: 2.2u, symbol Device:C
- added C105, C106: 0.1u, symbol Device:C
- added R102, R103: 1k, symbol Device:R
- renumbered J101 to MAG_ENABLE_OUT101
Connections:
- net +5VIN: now also C101.1, C107.1, C108.1
- net +5VOut1: now also C104.1, C106.2
- net +5VOut2: now also C103.1
- net GND: now also C103.2, C104.2, C106.1, R102.1, R103.1; no longer U101.11 (B4), U101.12 (B3)
- net PWR_GND_IN: now also C101.2, C107.2, C108.2
- net at U101.1 (VDD1), VT101.8 (+VOUT): now also C102.1, C105.1
- net at ERR_In101.2 (BNC_Shield), ERR_In101.3 (shield), ERR_In101.4 (shield)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: now also C102.2, C105.2
- new net: R103.2, U101.11 (B4)
- new net: R102.2, U101.12 (B3)

Commit message: Adding Footprints
Parts:
- C101, C102, C103, C104, C105, C106, C107, C108: footprint (none) -> Capacitor_SMD:C_1206_3216Metric_Pad1.42x1.75mm_HandSolder
- ERR_In101, MAG_ENABLE_OUT101: footprint conn2_1-1337543-0_TEC -> BNC_female:1-1337543-0
- PWR_In101: footprint 691508110303 -> 3PinPowerTerm:691508110303
- R101, R102, R103: footprint (none) -> Resistor_SMD:R_1206_3216Metric_Pad1.42x1.75mm_HandSolder
- S101: footprint CL-SB-12B -> CL-SB-12B-01T:CL-SB-12B
- U101: footprint SOIC-16W_SIL -> SI8640DBIS:Si8640BD-B-IS
- VT101, VT102, VT103: footprint VREG_NXJ1S0505MC-R7 -> NXJ1S050:VREG_NXJ1S0505MC-R7
Changed lines of the file:
@@
 F 0 "U101" H 5250 1487 60  0000 C CNN
 F 1 "Si8640BD-B-IS" H 5250 1381 60  0000 C CNN
-F 2 "SOIC-16W_SIL" H 5250 1340 60  0001 C CNN
+F 2 "SI8640DBIS:Si8640BD-B-IS" H 5250 1340 60  0001 C CNN
 F 3 "" H 4050 1100 60  0000 C CNN
 	1    4050 1100
@@
 F 0 "PWR_In101" H 943 1867 50  0000 C CNN
 F 1 "691508110303" H 943 1776 50  0000 C CNN
-F 2 "691508110303" H 1000 1500 50  0001 L BNN
+F 2 "3PinPowerTerm:691508110303" H 1000 1500 50  0001 L BNN
 F 3 "" H 1000 1500 50  0001 C CNN
 	1    1000 1500
@@
 F 0 "VT101" H 1800 1925 50  0000 C CNN
 F 1 "NXJ1S0505MC-R7" H 1800 1834 50  0000 C CNN
-F 2 "VREG_NXJ1S0505MC-R7" H 1350 1800 50  0001 L BNN
+F 2 "NXJ1S050:VREG_NXJ1S0505MC-R7" H 1350 1800 50  0001 L BNN
 F 3 "muRata" H 1800 2200 50  0001 L BNN
 	1    1800 2200
@@
 F 0 "VT102" H 1800 2875 50  0000 C CNN
 F 1 "NXJ1S0505MC-R7" H 1800 2784 50  0000 C CNN
-F 2 "VREG_NXJ1S0505MC-R7" H 1350 2750 50  0001 L BNN
+F 2 "NXJ1S050:VREG_NXJ1S0505MC-R7" H 1350 2750 50  0001 L BNN
 F 3 "muRata" H 1800 3150 50  0001 L BNN
 	1    1800 3150
@@
 F 0 "VT103" H 1800 3825 50  0000 C CNN
 F 1 "NXJ1S0505MC-R7" H 1800 3734 50  0000 C CNN
-F 2 "VREG_NXJ1S0505MC-R7" H 1350 3700 50  0001 L BNN
+F 2 "NXJ1S050:VREG_NXJ1S0505MC-R7" H 1350 3700 50  0001 L BNN
 F 3 "muRata" H 1800 4100 50  0001 L BNN
 	1    1800 4100
@@
 F 0 "ERR_In101" H 3542 1637 60  0000 C CNN
 F 1 "BNC_Input_female" H 3542 1531 60  0000 C CNN
-F 2 "conn2_1-1337543-0_TEC" H 3700 1290 60  0001 C CNN
+F 2 "BNC_female:1-1337543-0" H 3700 1290 60  0001 C CNN
 F 3 "" H 3300 1350 60  0000 C CNN
 	1    3300 1350
@@
 F 0 "S101" H 7900 1127 50  0000 C CNN
 F 1 "CL-SB-12B-01T" H 7900 1036 50  0000 C CNN
-F 2 "CL-SB-12B" H 7900 1400 50  0001 L BNN
+F 2 "CL-SB-12B-01T:CL-SB-12B" H 7900 1400 50  0001 L BNN
 F 3 "" H 7900 1400 50  0001 C CNN
 	1    7900 1400
@@
 F 0 "R101" H 7970 896 50  0000 L CNN
 F 1 "10k" H 7970 805 50  0000 L CNN
-F 2 "" V 7830 850 50  0001 C CNN
+F 2 "Resistor_SMD:R_1206_3216Metric_Pad1.42x1.75mm_HandSolder" V 7830 850 50  0001 C CNN
 F 3 "~" H 7900 850 50  0001 C CNN
 	1    7900 850
@@
 F 0 "MAG_ENABLE_OUT101" H 8628 3353 60  0000 L CNN
 F 1 "BNC_Input_female" H 8628 3247 60  0000 L CNN
-F 2 "conn2_1-1337543-0_TEC" H 8500 3390 60  0001 C CNN
+F 2 "BNC_female:1-1337543-0" H 8500 3390 60  0001 C CNN
 F 3 "" H 8100 3450 60  0000 C CNN
 	1    8100 3450
@@
 F 0 "C107" V 1352 2850 50  0000 C CNN
 F 1 "4.7u" V 1261 2850 50  0000 C CNN
-F 2 "" H 1138 2700 50  0001 C CNN
+F 2 "Capacitor_SMD:C_1206_3216Metric_Pad1.42x1.75mm_HandSolder" H 1138 2700 50  0001 C CNN
 F 3 "~" H 1100 2850 50  0001 C CNN
 	1    1100 2850
@@
 F 0 "C101" V 1402 1950 50  0000 C CNN
 F 1 "4.7u" V 1311 1950 50  0000 C CNN
-F 2 "" H 1188 1800 50  0001 C CNN
+F 2 "Capacitor_SMD:C_1206_3216Metric_Pad1.42x1.75mm_HandSolder" H 1188 1800 50  0001 C CNN
 F 3 "~" H 1150 1950 50  0001 C CNN
 	1    1150 1950
@@
 F 0 "C108" V 1402 3850 50  0000 C CNN
 F 1 "4.7u" V 1311 3850 50  0000 C CNN
-F 2 "" H 1188 3700 50  0001 C CNN
+F 2 "Capacitor_SMD:C_1206_3216Metric_Pad1.42x1.75mm_HandSolder" H 1188 3700 50  0001 C CNN
 F 3 "~" H 1150 3850 50  0001 C CNN
 	1    1150 3850
@@
 F 0 "C105" V 3648 800 50  0000 C CNN
 F 1 "0.1u" V 3739 800 50  0000 C CNN
-F 2 "" H 3938 650 50  0001 C CNN
+F 2 "Capacitor_SMD:C_1206_3216Metric_Pad1.42x1.75mm_HandSolder" H 3938 650 50  0001 C CNN
 F 3 "~" H 3900 800 50  0001 C CNN
 	1    3900 800
@@
 F 0 "C106" V 6248 750 50  0000 C CNN
 F 1 "0.1u" V 6339 750 50  0000 C CNN
-F 2 "" H 6538 600 50  0001 C CNN
+F 2 "Capacitor_SMD:C_1206_3216Metric_Pad1.42x1.75mm_HandSolder" H 6538 600 50  0001 C CNN
 F 3 "~" H 6500 750 50  0001 C CNN
 	1    6500 750
@@
 F 0 "C102" V 2902 2100 50  0000 C CNN
 F 1 "2.2u" V 2811 2100 50  0000 C CNN
-F 2 "" H 2688 1950 50  0001 C CNN
+F 2 "Capacitor_SMD:C_1206_3216Metric_Pad1.42x1.75mm_HandSolder" H 2688 1950 50  0001 C CNN
 F 3 "~" H 2650 2100 50  0001 C CNN
 	1    2650 2100
@@
 F 0 "C104" H 3415 3246 50  0000 L CNN
 F 1 "2.2u" H 3415 3155 50  0000 L CNN
-F 2 "" H 3338 3050 50  0001 C CNN
+F 2 "Capacitor_SMD:C_1206_3216Metric_Pad1.42x1.75mm_HandSolder" H 3338 3050 50  0001 C CNN
 F 3 "~" H 3300 3200 50  0001 C CNN
 	1    3300 3200
@@
 F 0 "C103" H 3365 4196 50  0000 L CNN
 F 1 "2.2u" H 3365 4105 50  0000 L CNN
-F 2 "" H 3288 4000 50  0001 C CNN
+F 2 "Capacitor_SMD:C_1206_3216Metric_Pad1.42x1.75mm_HandSolder" H 3288 4000 50  0001 C CNN
 F 3 "~" H 3250 4150 50  0001 C CNN
 	1    3250 4150
@@
 F 0 "R102" V 6493 1500 50  0000 C CNN
 F 1 "1k" V 6584 1500 50  0000 C CNN
-F 2 "" V 6630 1500 50  0001 C CNN
+F 2 "Resistor_SMD:R_1206_3216Metric_Pad1.42x1.75mm_HandSolder" V 6630 1500 50  0001 C CNN
 F 3 "~" H 6700 1500 50  0001 C CNN
 	1    6700 1500
@@
 F 0 "R103" V 6493 1600 50  0000 C CNN
 F 1 "1k" V 6584 1600 50  0000 C CNN
-F 2 "" V 6630 1600 50  0001 C CNN
+F 2 "Resistor_SMD:R_1206_3216Metric_Pad1.42x1.75mm_HandSolder" V 6630 1600 50  0001 C CNN
 F 3 "~" H 6700 1600 50  0001 C CNN
 	1    6700 1600

Commit message: Enrique changes
Parts:
- removed C101: 4.7u, Capacitor_SMD:C_1206_3216Metric_Pad1.42x1.75mm_HandSolder, symbol Device:C
- removed C102: 2.2u, Capacitor_SMD:C_1206_3216Metric_Pad1.42x1.75mm_HandSolder, symbol Device:C
- removed MAG_ENABLE_OUT101: BNC_Input_female, BNC_female:1-1337543-0, symbol magnets_interlock_library:BNC_Input_female
- removed VT101: NXJ1S0505MC-R7, NXJ1S050:VREG_NXJ1S0505MC-R7, symbol NXJ1S0505MC-R7:NXJ1S0505MC-R7
- added C109: 47u, Capacitor_THT:CP_Radial_D8.0mm_P3.50mm, symbol Device:C
- added C110, C111: 4.7u, Capacitor_SMD:C_1206_3216Metric_Pad1.42x1.75mm_HandSolder, symbol Device:C
Connections:
- net +5VIN: now also C105.1, U101.1 (VDD1), C109.2, C110.2, C111.2
- net PWR_GND_IN: now also C105.2, ERR_In101.2 (BNC_Shield), ERR_In101.3 (shield), ERR_In101.4 (shield), U101.2 (GND1), U101.5 (A3), U101.6 (A4), U101.8 (GND1), C109.1, C110.1, C111.1
Changed lines of the file:
@@
 U 1 1 5EF7A439
 P 1000 1500
-F 0 "PWR_In101" H 943 1867 50  0000 C CNN
-F 1 "691508110303" H 943 1776 50  0000 C CNN
+F 0 "PWR_In101" H 1100 1850 50  0000 C CNN
+F 1 "691508110303" H 1050 1750 50  0000 C CNN
 F 2 "3PinPowerTerm:691508110303" H 1000 1500 50  0001 L BNN
 F 3 "" H 1000 1500 50  0001 C CNN
@@
 +5VIN
 Wire Wire Line
-	1450 1400 1250 1400
+	1450 1400 1400 1400
 Text GLabel 1450 1600 2    50   Input ~ 0
 PWR_GND_IN
@@
 	1450 1600 1250 1600
 NoConn ~ 1250 1500
-$Comp
-L NXJ1S0505MC-R7:NXJ1S0505MC-R7 VT101
-U 1 1 5EF9CB9B
-P 1800 2200
-AR Path="/5EF9CB9B" Ref="VT101"  Part="1"
-AR Path="/5EF82676/5EF9CB9B" Ref="VT?"  Part="1"
-F 0 "VT101" H 1800 1925 50  0000 C CNN
-F 1 "NXJ1S0505MC-R7" H 1800 1834 50  0000 C CNN
-F 2 "NXJ1S050:VREG_NXJ1S0505MC-R7" H 1350 1800 50  0001 L BNN
-F 3 "muRata" H 1800 2200 50  0001 L BNN
-	1    1800 2200
-	1    0    0    -1
-$EndComp
 $Comp
 L NXJ1S0505MC-R7:NXJ1S0505MC-R7 VT102
@@
 	1    0    0    -1
 $EndComp
-Text GLabel 950  2100 0    50   Input ~ 0
-+5VIN
 Text GLabel 950  3050 0    50   Input ~ 0
 +5VIN
 Text GLabel 950  4000 0    50   Input ~ 0
 +5VIN
-Text GLabel 1050 2300 0    50   Input ~ 0
-PWR_GND_IN
 Text GLabel 1050 3250 0    50   Input ~ 0
 PWR_GND_IN
 Text GLabel 1050 4200 0    50   Input ~ 0
 PWR_GND_IN
-Wire Wire Line
-	950  2100 1050 2100
-Wire Wire Line
-	1050 2300 1150 2300
 Wire Wire Line
 	950  3050 1050 3050
@@
 Wire Wire Line
 	4000 1800 4050 1800
-Wire Wire Line
-	3800 2300 3800 1800
-Wire Wire Line
-	3800 1800 3900 1800
 Connection ~ 3900 1800
-Wire Wire Line
-	2400 2100 2400 900
-Wire Wire Line
-	2400 900  3550 900
 Wire Wire Line
 	3550 900  3550 1100
@@
 	7250 1000 7900 1000
 Connection ~ 7900 1000
-$Comp
-L magnets_interlock_library:BNC_Input_female MAG_ENABLE_OUT101
-U 1 1 5EFC2490
-P 8100 3450
-F 0 "MAG_ENABLE_OUT101" H 8628 3353 60  0000 L CNN
-F 1 "BNC_Input_female" H 8628 3247 60  0000 L CNN
-F 2 "BNC_female:1-1337543-0" H 8500 3390 60  0001 C CNN
-F 3 "" H 8100 3450 60  0000 C CNN
-	1    8100 3450
-	1    0    0    -1
-$EndComp
 $Sheet
 S 4300 4650 2750 950
@@
 Wire Wire Line
 	3950 5050 4300 5050
-Wire Wire Line
-	8100 3650 8100 3700
-$Comp
-L power:GND #PWR0114
-U 1 1 5EFD2B4D
-P 7850 3700
-F 0 "#PWR0114" H 7850 3450 50  0001 C CNN
-F 1 "GND" H 7855 3527 50  0000 C CNN
-F 2 "" H 7850 3700 50  0001 C CNN
-F 3 "" H 7850 3700 50  0001 C CNN
-	1    7850 3700
-	1    0    0    -1
-$EndComp
-Wire Wire Line
-	7850 3700 8100 3700
-Connection ~ 8100 3700
-Wire Wire Line
-	8100 3700 8100 3750
 $Sheet
 S 4350 2950 2650 1250
@@
 $EndComp
 $Comp
-L Device:C C101
-U 1 1 5EFF9CF9
-P 1150 1950
-F 0 "C101" V 1402 1950 50  0000 C CNN
-F 1 "4.7u" V 1311 1950 50  0000 C CNN
-F 2 "Capacitor_SMD:C_1206_3216Metric_Pad1.42x1.75mm_HandSolder" H 1188 1800 50  0001 C CNN
-F 3 "~" H 1150 1950 50  0001 C CNN
-	1    1150 1950
-	0    -1   -1   0
-$EndComp
-$Comp
 L Device:C C108
 U 1 1 5EFFA3CD
@@
 $EndComp
 Wire Wire Line
-	1000 1950 1000 2050
-Wire Wire Line
-	1000 2050 1050 2050
-Wire Wire Line
-	1050 2050 1050 2100
-Connection ~ 1050 2100
-Wire Wire Line
-	1050 2100 1200 2100
-Wire Wire Line
-	1300 1950 1300 2050
-Wire Wire Line
-	1300 2050 1150 2050
-Wire Wire Line
-	1150 2050 1150 2300
-Connection ~ 1150 2300
-Wire Wire Line
-	1150 2300 1200 2300
-Wire Wire Line
 	950  2850 950  2950
 Wire Wire Line
@@
 	6650 750  6650 1000
 $Comp
-L Device:C C102
-U 1 1 5F018AC0
-P 2650 2100
-F 0 "C102" V 2902 2100 50  0000 C CNN
-F 1 "2.2u" V 2811 2100 50  0000 C CNN
-F 2 "Capacitor_SMD:C_1206_3216Metric_Pad1.42x1.75mm_HandSolder" H 2688 1950 50  0001 C CNN
-F 3 "~" H 2650 2100 50  0001 C CNN
-	1    2650 2100
-	0    -1   -1   0
-$EndComp
-Wire Wire Line
-	2500 2100 2400 2100
-Connection ~ 2400 2100
-$Comp
 L Device:C C104
 U 1 1 5F023665
@@
 Wire Wire Line
 	2850 3350 2850 3250
-Wire Wire Line
-	2400 2300 2800 2300
-Wire Wire Line
-	2800 2100 2800 2300
-Connection ~ 2800 2300
-Wire Wire Line
-	2800 2300 3800 2300
 Wire Wire Line
 	6450 1800 6700 1800
@@
 Wire Wire Line
 	7000 1550 7000 2000
+$Comp
+L Device:C C109
+U 1 1 5F0C5580
+P 1400 1000
+F 0 "C109" H 1515 1046 50  0000 L CNN
+F 1 "47u" H 1515 955 50  0000 L CNN
+F 2 "Capacitor_THT:CP_Radial_D8.0mm_P3.50mm" H 1438 850 50  0001 C CNN
+F 3 "~" H 1400 1000 50  0001 C CNN
+	1    1400 1000
+	1    0    0    -1
+$EndComp
+Connection ~ 1400 1400
+Wire Wire Line
+	1400 1400 1250 1400
+Text GLabel 1400 650  2    50   Input ~ 0
+PWR_GND_IN
+$Comp
+L Device:C C110
+U 1 1 5F0D1FE9
+P 1150 1000
+F 0 "C110" H 1265 1046 50  0000 L CNN
+F 1 "4.7u" H 1265 955 50  0000 L CNN
+F 2 "Capacitor_SMD:C_1206_3216Metric_Pad1.42x1.75mm_HandSolder" H 1188 850 50  0001 C CNN
+F 3 "~" H 1150 1000 50  0001 C CNN
+	1    1150 1000
+	1    0    0    -1
+$EndComp
+$Comp
+L Device:C C111
+U 1 1 5F0D256B
+P 1800 1050
+F 0 "C111" H 1915 1096 50  0000 L CNN
+F 1 "4.7u" H 1915 1005 50  0000 L CNN
+F 2 "Capacitor_SMD:C_1206_3216Metric_Pad1.42x1.75mm_HandSolder" H 1838 900 50  0001 C CNN
+F 3 "~" H 1800 1050 50  0001 C CNN
+	1    1800 1050
+	1    0    0    -1
+$EndComp
+Wire Wire Line
+	1800 1200 1400 1200
+Wire Wire Line
+	1400 1150 1400 1200
+Connection ~ 1400 1200
+Wire Wire Line
+	1400 1200 1400 1400
+Wire Wire Line
+	1400 1200 1150 1200
+Wire Wire Line
+	1150 1200 1150 1150
+Wire Wire Line
+	1150 850  1150 800
+Wire Wire Line
+	1150 800  1400 800
+Connection ~ 1400 800
+Wire Wire Line
+	1400 800  1400 850
+Wire Wire Line
+	1800 900  1800 800
+Wire Wire Line
+	1800 800  1400 800
+Wire Wire Line
+	1400 650  1400 800
+Text GLabel 3700 1800 0    50   Input ~ 0
+PWR_GND_IN
+Wire Wire Line
+	3700 1800 3900 1800
+Text GLabel 2950 900  0    50   Input ~ 0
++5VIN
+Wire Wire Line
+	2950 900  3550 900
 $EndSCHEMATC

Commit message: Draft 1 Almost There
Parts:
- removed C108: 4.7u, Capacitor_SMD:C_1206_3216Metric_Pad1.42x1.75mm_HandSolder, symbol Device:C
- removed C109: 47u, Capacitor_THT:CP_Radial_D8.0mm_P3.50mm, symbol Device:C
- removed U101: Si8640BD-B-IS, SI8640DBIS:Si8640BD-B-IS, symbol 2020-06-26_17-59-50:Si8640BD-B-IS
- removed VT103: NXJ1S0505MC-R7, NXJ1S050:VREG_NXJ1S0505MC-R7, symbol NXJ1S0505MC-R7:NXJ1S0505MC-R7
- added C101: 0.1u, Capacitor_SMD:C_1206_3216Metric_Pad1.42x1.75mm_HandSolder, symbol Device:C
- added C102: 2.2u, Capacitor_SMD:C_1206_3216Metric_Pad1.42x1.75mm_HandSolder, symbol Device:C
- added C109: 47u, Capacitor_THT:CP_Radial_D8.0mm_P3.50mm, symbol Device:CP1
- added L101, L103: 4.7u, VLCF4024T-4R7N1R4-2:VLCF4024T-4R7N1R4-2, symbol 2020-06-30_20-16-32:VLCF4024T-4R7N1R4-2
- added L102, L104: 10u, VLCF4024T-4R7N1R4-2:VLCF4024T-4R7N1R4-2, symbol 2020-06-30_19-50-11:VLCF4024T-100MR90-2
- added Relay_Off_Output101: BNC_Input_female, BNC_female:1-1337543-0, symbol magnets_interlock_library:BNC_Input_female
- added S102: CL-SB-12B-01T, CL-SB-12B-01T:CL-SB-12B, symbol CL-SB-12B-01T:CL-SB-12B-01T
- added U101: ISO7741FDWR, ISO7741FDWR:ISO7741FDWR, symbol 2020-06-30_17-30-58:ISO7741FDWR
- added U102: SN74LVC1G08DCKR, inverter:SN74LVC1G14DCKR, symbol dk_Logic-Gates-and-Inverters:SN74LVC1G08DCKR
- added U103: 691321100003, Magnet_PS_Interlock:691321100003, symbol enrique_3termscrew:691321100003
- added VT101: NXJ1S0505MC-R7, NXJ1S050:VREG_NXJ1S0505MC-R7, symbol NXJ1S0505MC-R7:NXJ1S0505MC-R7
- C103: value 2.2u -> 4.7u
- R102, R103: value 1k -> 10k
Connections:
- net +5VIN: now also C103.1, C109.1, L101.2, L103.2, S102.1, U101.1 (VCC1); no longer VT102.3 (+VIN)
- net +5VOut1: now also C102.1, L102.1, U101.16 (VCC2); no longer C104.1, VT102.8 (+VOUT)
- net +5VOut2: now also C104.1, C101.2, L104.1, U102.5 (VCC); no longer C103.1
- net GND: now also C101.1, C102.2, U101.15 (GND2), U101.9 (GND2), U102.3 (GND), VT101.7 (-VOUT); no longer C103.2, R103.1
- net PWR_GND_IN: now also C103.2, R103.1, C109.2, Relay_Off_Output101.2 (BNC_Shield), Relay_Off_Output101.3 (shield), Relay_Off_Output101.4 (shield), S102.3, U101.2 (GND1), U101.5 (INC), U101.8 (GND1), VT101.1 (-VIN)
- net Relay_1/Enable_Conn_1: now also U103.3
- net Relay_1/ErrSig1: now also U101.14 (OUTA)
- net Relay_2/Enable_Conn_2: now also U103.2
- net Relay_2/ErrSig1: now also U101.13 (OUTB)
- net at R101.2, S101.2: now also U101.10 (EN2)
- net at R103.2: now also S102.2, U101.7 (EN1)
- net at R102.2: now also U101.12 (OUTC)
- net at ERR_In101.1 (Center_Pin): now also U101.3 (INA), U101.4 (INB)
- new net: L101.1, VT102.3 (+VIN)
- new net: L102.2, VT102.8 (+VOUT)
- new net: L104.2, VT101.8 (+VOUT)
- new net: L103.1, VT101.3 (+VIN)
- new net: Relay_Off_Output101.1 (Center_Pin), U101.6 (OUTD)
- new net Relay_1/Relay-Off-Sig: U102.1 (A)
- new net Relay_2/Relay-Off-Sig: U102.2 (B)
- new net Relay_off_signal: U101.11 (IND), U102.4 (Y)
- no-connect marks 1 -> 2
Other:
- moved on the sheet: C107, C110, C111, PWR_In101, R101, VT102
